File: hardware/drive/R2D2-drive.kicad_pcb (KiCad board)
At the start: 2 copper layers, 95 x 55 mm, 53 parts, among them J1 1751248, J2 1751248, J3 1751248, J4 1935776, J5 1935776, J6 Conn_01x05_Pin, SW1 PTS636 SM50J SMTR LFS, U1 LM1117MP-3.3, U2 STM32F042F6Px, U3 SN65HVD230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

Commit message: hw: drive: added a solder jumper for CAN address
Parts:
- added JP1: CAN_address, Jumper:SolderJumper-2_P1.3mm_Open_TrianglePad1.0x1.5mm, F.Cu at (126.2, 97.8)
- R10, R12: value ~ -> 5k1
- R11, R13: value ~ -> 1k
Connections:
- U2 pad 14: unconnected-(U2-PB1-Pad14) -> Net-(JP1-B)
Routing:
- net Net-(JP1-B): track 0.00 -> 8.24 mm
Other:
- board text added: "V1.1"
- board text added: "march 2025"
- board text removed: "V1"
- board text removed: "october 2024"
