File: hardware/battery-control/power_stage.kicad_sch (KiCad schematic)
At the start: 18 parts, among them J4 1935776, J5 1935776, K1 J123F1C12VDC.36, Q1 T2N7002AK, U3 TPS62172DSGR, U4 LM321

Commit message: hw: battery-control: R6 should not be populated. The internal resistors of MCU are used instead
Parts:
- R6: now not fitted
Changed lines of the file:
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@@
 (kicad_sch
-	(version 20231120)
+	(version 20250114)
 	(generator "eeschema")
-	(generator_version "8.0")
+	(generator_version "9.0")
 	(paper "A4")
 	(junction
@@
 		(in_bom yes)
 		(on_board yes)
-		(dnp no)
+		(dnp yes)
 		(property "Reference" "R6"
 			(at 228.6 99.06 90)
